File: MPE_HUB_Board/HUB_MPE.kicad_sch (KiCad schematic)
At the start: 18 parts, among them J1 Conn_01x09, J2 Conn_01x03, J3 Conn_01x06, J4 Conn_01x07, J5 Conn_01x05, J6 Conn_01x05, U1 K7803M-1000R3_C2916516

Commit message: Risolto problema reset (Nel firmware V2)
Parts:
- J2: footprint Connector_JST:JST_EH_B3B-EH-A_1x03_P2.50mm_Vertical -> Connector_JST:JST_VH_B3P-VH_1x03_P3.96mm_Vertical
- J3: footprint Connector_JST:JST_EH_B6B-EH-A_1x06_P2.50mm_Vertical -> Connector_JST:JST_VH_B6P-VH-B_1x06_P3.96mm_Vertical
- J4: footprint Connector_JST:JST_EH_B7B-EH-A_1x07_P2.50mm_Vertical -> Connector_JST:JST_VH_B7P-VH-B_1x07_P3.96mm_Vertical
Connections:
- net 485_ROV+: no longer J5.2 (Pin_2), J6.2 (Pin_2)
- net 485_ROV-: no longer J5.3 (Pin_3), J6.3 (Pin_3)
- new net 485_LED+: J5.2 (Pin_2), J6.2 (Pin_2)
- new net 485_LED-: J5.3 (Pin_3), J6.3 (Pin_3)
Other:
- sheet MCU_ESP32 ports: added 485_LED_A, 485_LED_B, 485_ROV_A, 485_ROV_B; removed 485A, 485B
Changed lines of the file:
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@@
 	(title_block
 		(title "HUB_MPE")
-		(date "2025-03-24")
+		(date "2025-03-21")
 		(rev "0.1")
 		(company "3DResearch")
@@
 	(wire
 		(pts
+			(xy 325.12 217.17) (xy 345.44 217.17)
+		)
+		(stroke
+			(width 0)
+			(type default)
+		)
+	)
+	(wire
+		(pts
 			(xy 149.86 176.53) (xy 130.81 176.53)
 		)
@@
 	(wire
 		(pts
-			(xy 341.63 50.8) (xy 339.09 50.8)
+			(xy 345.44 193.04) (xy 325.12 193.04)
 		)
 		(stroke
@@
 	(wire
 		(pts
-			(xy 226.06 132.08) (xy 245.11 132.08)
+			(xy 341.63 50.8) (xy 339.09 50.8)
 		)
 		(stroke
@@
 	(wire
 		(pts
-			(xy 38.1 30.48) (xy 38.1 33.02)
+			(xy 226.06 132.08) (xy 245.11 132.08)
 		)
 		(stroke
@@
 	(wire
 		(pts
-			(xy 57.15 63.5) (xy 58.42 63.5)
+			(xy 38.1 30.48) (xy 38.1 33.02)
 		)
 		(stroke
@@
 	(wire
 		(pts
-			(xy 345.44 127) (xy 325.12 127)
+			(xy 57.15 63.5) (xy 58.42 63.5)
 		)
 		(stroke
@@
 	(wire
 		(pts
-			(xy 149.86 228.6) (xy 130.81 228.6)
+			(xy 345.44 219.71) (xy 325.12 219.71)
 		)
 		(stroke
@@
 	(wire
 		(pts
-			(xy 71.12 38.1) (xy 80.01 38.1)
+			(xy 345.44 127) (xy 325.12 127)
 		)
 		(stroke
@@
 	(wire
 		(pts
-			(xy 345.44 113.03) (xy 326.39 113.03)
+			(xy 149.86 228.6) (xy 130.81 228.6)
 		)
 		(stroke
@@
 	(wire
 		(pts
-			(xy 345.44 193.04) (xy 325.12 193.04)
+			(xy 71.12 38.1) (xy 80.01 38.1)
 		)
 		(stroke
@@
 	(wire
 		(pts
-			(xy 350.52 53.34) (xy 347.98 53.34)
+			(xy 345.44 113.03) (xy 326.39 113.03)
 		)
 		(stroke
@@
 	(wire
 		(pts
-			(xy 345.44 214.63) (xy 325.12 214.63)
+			(xy 350.52 53.34) (xy 347.98 53.34)
 		)
 		(stroke
@@
 	(wire
 		(pts
-			(xy 217.17 219.71) (xy 217.17 220.98)
+			(xy 345.44 214.63) (xy 325.12 214.63)
 		)
 		(stroke
@@
 	(wire
 		(pts
-			(xy 345.44 217.17) (xy 325.12 217.17)
+			(xy 217.17 219.71) (xy 217.17 220.98)
 		)
 		(stroke
@@
 	(wire
 		(pts
+			(xy 149.86 212.09) (xy 130.81 212.09)
+		)
+		(stroke
+			(width 0)
+			(type default)
+		)
+	)
+	(wire
+		(pts
 			(xy 203.2 226.06) (xy 220.98 226.06)
 		)
@@
 	(wire
 		(pts
-			(xy 345.44 190.5) (xy 325.12 190.5)
-		)
-		(stroke
-			(width 0)
-			(type default)
-		)
-	)
-	(wire
-		(pts
 			(xy 330.2 60.96) (xy 350.52 60.96)
 		)
@@
 	(wire
 		(pts
-			(xy 345.44 219.71) (xy 325.12 219.71)
+			(xy 203.2 209.55) (xy 220.98 209.55)
 		)
 		(stroke
@@
 	(wire
 		(pts
-			(xy 203.2 209.55) (xy 220.98 209.55)
+			(xy 226.06 121.92) (xy 245.11 121.92)
 		)
 		(stroke
@@
 	(wire
 		(pts
-			(xy 226.06 121.92) (xy 245.11 121.92)
+			(xy 341.63 46.99) (xy 341.63 50.8)
 		)
 		(stroke
@@
 	(wire
 		(pts
-			(xy 341.63 46.99) (xy 341.63 50.8)
+			(xy 203.2 223.52) (xy 220.98 223.52)
 		)
 		(stroke
@@
 	(wire
 		(pts
-			(xy 203.2 223.52) (xy 220.98 223.52)
+			(xy 80.01 38.1) (xy 80.01 39.37)
 		)
 		(stroke
@@
 	(wire
 		(pts
-			(xy 80.01 38.1) (xy 80.01 39.37)
+			(xy 325.12 190.5) (xy 345.44 190.5)
 		)
 		(stroke
@@
 	(wire
 		(pts
+			(xy 149.86 209.55) (xy 130.81 209.55)
+		)
+		(stroke
+			(width 0)
+			(type default)
+		)
+	)
+	(wire
+		(pts
 			(xy 52.07 33.02) (xy 82.55 33.02)
 		)
@@
 		)
 	)
-	(label "485_ROV+"
-		(at 325.12 190.5 0)
-		(effects
-			(font
-				(size 1.27 1.27)
-			)
-			(justify left bottom)
-		)
-	)
 	(label "RESET_SWITCH"
 		(at 130.81 228.6 0)
@@
 		)
 	)
-	(label "485_ROV+"
-		(at 325.12 217.17 0)
-		(effects
-			(font
-				(size 1.27 1.27)
-			)
-			(justify left bottom)
-		)
-	)
 	(label "ETH_BD3D_TX-"
 		(at 245.11 105.41 180)
@@
 		)
 	)
+	(label "485_LED+"
+		(at 325.12 217.17 0)
+		(effects
+			(font
+				(size 1.27 1.27)
+			)
+			(justify left bottom)
+		)
+	)
 	(label "+24V_FLASH1"
 		(at 278.13 201.93 180)
@@
 		)
 	)
-	(label "485_ROV-"
-		(at 325.12 219.71 0)
-		(effects
-			(font
-				(size 1.27 1.27)
-			)
-			(justify left bottom)
-		)
-	)
 	(label "ETH_IPCAM_TX+"
 		(at 171.45 102.87 0)
@@
 		)
 	)
-	(label "485_ROV-"
-		(at 325.12 193.04 0)
+	(label "+24V_FLASH2"
+		(at 278.13 207.01 180)
 		(effects
 			(font
 				(size 1.27 1.27)
 			)
-			(justify left bottom)
+			(justify right bottom)
 		)
 	)
-	(label "+24V_FLASH2"
-		(at 278.13 207.01 180)
+	(label "485_LED-"
+		(at 130.81 212.09 0)
 		(effects
 			(font
 				(size 1.27 1.27)
 			)
-			(justify right bottom)
+			(justify left bottom)
 		)
 	)
@@
 		)
 	)
+	(label "485_LED-"
+		(at 325.12 219.71 0)
+		(effects
+			(font
+				(size 1.27 1.27)
+			)
+			(justify left bottom)
+		)
+	)
 	(label "ETH_ESP_TX-"
 		(at 245.11 116.84 180)
@@
 		)
 	)
+	(label "485_LED+"
+		(at 325.12 190.5 0)
+		(effects
+			(font
+				(size 1.27 1.27)
+			)
+			(justify left bottom)
+		)
+	)
 	(label "485_ROV-"
 		(at 350.52 68.58 180)
@@
 		)
 	)
+	(label "485_LED-"
+		(at 325.12 193.04 0)
+		(effects
+			(font
+				(size 1.27 1.27)
+			)
+			(justify left bottom)
+		)
+	)
 	(label "EXPOSURE"
 		(at 325.12 222.25 0)
@@
 		)
 	)
+	(label "485_LED+"
+		(at 130.81 209.55 0)
+		(effects
+			(font
+				(size 1.27 1.27)
+			)
+			(justify left bottom)
+		)
+	)
 	(label "ETH_BD3D_TX+"
 		(at 325.12 153.67 0)
@@
 		(polyline
 			(pts
-				(xy 186.055 97.79) (xy 187.325 97.79) (xy 187.325 124.46) (xy 186.055 124.46)
+				(xy 227.965 97.79) (xy 229.235 97.79) (xy 229.235 124.46) (xy 227.965 124.46)
 			)
 			(stroke
@@
 		(polyline
 			(pts
-				(xy 227.965 97.79) (xy 229.235 97.79) (xy 229.235 124.46) (xy 227.965 124.46)
+				(xy 186.055 97.79) (xy 187.325 97.79) (xy 187.325 124.46) (xy 186.055 124.46)
 			)
 			(stroke
@@
 			)
 		)
-		(property "Footprint" "Connector_JST:JST_EH_B6B-EH-A_1x06_P2.50mm_Vertical"
+		(property "Footprint" "Connector_JST:JST_VH_B6P-VH-B_1x06_P3.96mm_Vertical"
 			(at 350.52 132.08 0)
 			(effects
@@
 			)
 		)
-		(property "Footprint" "Connector_JST:JST_EH_B3B-EH-A_1x03_P2.50mm_Vertical"
+		(property "Footprint" "Connector_JST:JST_VH_B3P-VH_1x03_P3.96mm_Vertical"
 			(at 350.52 110.49 0)
 			(effects
@@
 			)
 		)
-		(property "Footprint" "Connector_JST:JST_EH_B7B-EH-A_1x07_P2.50mm_Vertical"
+		(property "Footprint" "Connector_JST:JST_VH_B7P-VH-B_1x07_P3.96mm_Vertical"
 			(at 350.52 158.75 0)
 			(effects
@@
 			)
 		)
-		(pin "485A" bidirectional
-			(at 149.86 201.93 180)
-			(effects
-				(font
-					(size 1.27 1.27)
-				)
-				(justify left)
-			)
-		)
-		(pin "485B" bidirectional
-			(at 149.86 204.47 180)
-			(effects
-				(font
-					(size 1.27 1.27)
-				)
-				(justify left)
-			)
-		)
 		(pin "GND_MCU" input
 			(at 149.86 179.07 180)
@@
 			)
 		)
+		(pin "485_LED_A" bidirectional
+			(at 149.86 209.55 180)
+			(effects
+				(font
+					(size 1.27 1.27)
+				)
+				(justify left)
+			)
+		)
+		(pin "485_LED_B" bidirectional
+			(at 149.86 212.09 180)
+			(effects
+				(font
+					(size 1.27 1.27)
+				)
+				(justify left)
+			)
+		)
+		(pin "485_ROV_A" bidirectional
+			(at 149.86 201.93 180)
+			(effects
+				(font
+					(size 1.27 1.27)
+				)
+				(justify left)
+			)
+		)
+		(pin "485_ROV_B" bidirectional
+			(at 149.86 204.47 180)
+			(effects
+				(font
+					(size 1.27 1.27)
+				)
+				(justify left)
+			)
+		)

Commit message: Update 04/07/2025
Parts:
- removed LED2: 0805_RED, easyeda2kicad:LED0805-R-RD, symbol easyeda2kicad:FC-2012HRK-620D
- added LED2: 0805_YELLOW, easyeda2kicad:LED0805-R-RD, symbol easyeda2kicad:17-21SUYC_TR8
Connections:
- net GND: now also LED2.2 (-)
- net at R2.2: now also LED2.1 (+)
Other:
- sheet Power_Switch ports: added none; removed SE
- sheet Power_Switch1 ports: added none; removed SE
Changed lines of the file:
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@@
 	(wire
 		(pts
-			(xy 203.2 181.61) (xy 220.98 181.61)
-		)
-		(stroke
-			(width 0)
-			(type default)
-		)
-	)
-	(wire
-		(pts
 			(xy 330.2 55.88) (xy 350.52 55.88)
 		)
@@
 	(wire
 		(pts
-			(xy 203.2 209.55) (xy 220.98 209.55)
-		)
-		(stroke
-			(width 0)
-			(type default)
-		)
-	)
-	(wire
-		(pts
 			(xy 226.06 121.92) (xy 245.11 121.92)
 		)
@@
 	)
 	(symbol
+		(lib_id "easyeda2kicad:17-21SUYC_TR8")
+		(at 96.52 63.5 180)
+		(unit 1)
+		(exclude_from_sim no)
+		(in_bom yes)
+		(on_board yes)
+		(dnp no)
+		(property "Reference" "LED2"
+			(at 92.202 65.024 0)
+			(effects
+				(font
+					(size 1.27 1.27)
+				)
+			)
+		)
+		(property "Value" "0805_YELLOW"
+			(at 97.79 59.69 0)
+			(effects
+				(font
+					(size 1.27 1.27)
+				)
+			)
+		)
+		(property "Footprint" "easyeda2kicad:LED0805-R-RD"
+			(at 96.52 55.88 0)
+			(effects
+				(font
+					(size 1.27 1.27)
+				)
+				(hide yes)
+			)
+		)
+		(property "Datasheet" "https://lcsc.com/product-detail/Light-Emitting-Diodes-LED_Yellow-light-0805-Highlighted_C2296.html"
+			(at 96.52 53.34 0)
+			(effects
+				(font
+					(size 1.27 1.27)
+				)
+				(hide yes)
+			)
+		)
+		(property "Description" ""
+			(at 96.52 63.5 0)
+			(effects
+				(font
+					(size 1.27 1.27)
+				)
+				(hide yes)
+			)
+		)
+		(property "LCSC Part" "C2296"
+			(at 96.52 50.8 0)
+			(effects
+				(font
+					(size 1.27 1.27)
+				)
+				(hide yes)
+			)
+		)
+		(pin "1"
+		)
+		(pin "2"
+		)
+		(instances
+			(project ""
+				(path "/6490f62d-7c0a-4455-8633-837f094f0a1c"
+					(reference "LED2")
+					(unit 1)
+				)
+			)
+		)
+	)
+	(symbol
 		(lib_id "power:+24V")
 		(at 38.1 30.48 0)
@@
 	)
 	(symbol
-		(lib_id "easyeda2kicad:FC-2012HRK-620D")
-		(at 96.52 63.5 180)
-		(unit 1)
-		(exclude_from_sim no)
-		(in_bom yes)
-		(on_board yes)
-		(dnp no)
-		(property "Reference" "LED2"
-			(at 95.25 64.77 0)
-			(effects
-				(font
-					(size 1.27 1.27)
-				)
-				(justify left)
-			)
-		)
-		(property "Value" "0805_RED"
-			(at 101.854 59.944 0)
-			(effects
-				(font
-					(size 1.27 1.27)
-				)
-				(justify left)
-			)
-		)
-		(property "Footprint" "easyeda2kicad:LED0805-R-RD"
-			(at 96.52 55.88 0)
-			(effects
-				(font
-					(size 1.27 1.27)
-				)
-				(hide yes)
-			)
-		)
-		(property "Datasheet" "https://lcsc.com/product-detail/Light-Emitting-Diodes-LED_Red-LED-SMDLED-80-180mcd_C84256.html"
-			(at 96.52 53.34 0)
-			(effects
-				(font
-					(size 1.27 1.27)
-				)
-				(hide yes)
-			)
-		)
-		(property "Description" ""
-			(at 96.52 63.5 0)
-			(effects
-				(font
-					(size 1.27 1.27)
-				)
-				(hide yes)
-			)
-		)
-		(property "LCSC Part" "C84256"
-			(at 96.52 50.8 0)
-			(effects
-				(font
-					(size 1.27 1.27)
-				)
-				(hide yes)
-			)
-		)
-		(property "LCSC" "C84256"
-			(at 95.25 64.77 0)
-			(effects
-				(font
-					(size 1.27 1.27)
-				)
-				(hide yes)
-			)
-		)
-		(pin "2"
-		)
-		(pin "1"
-		)
-		(instances
-			(project "HUB_MPE"
-				(path "/6490f62d-7c0a-4455-8633-837f094f0a1c"
-					(reference "LED2")
-					(unit 1)
-				)
-			)
-		)
-	)
-	(symbol
 		(lib_id "Connector_Generic:Conn_01x05")
 		(at 350.52 193.04 0)
@@
 			)
 		)
-		(pin "SE" input
-			(at 220.98 209.55 180)
-			(effects
-				(font
-					(size 1.27 1.27)
-				)
-				(justify left)
-			)
-		)
 		(instances
 			(project "HUB_MPE"
@@
 			(effects
 				(font
-					(size 1.27 1.27)
-				)
-				(justify left)
-			)
-		)
-		(pin "SE" input
-			(at 220.98 181.61 180)
-			(effects
-				(font

Commit message: Update 08/07/2025
Parts:
- added TP4, TP5, TP6: TestPoint_Probe, easyeda2kicad:TEST-TH_BD2.54-P1.39, symbol Connector:TestPoint_Probe
Connections:
- net +24V: now also TP4.1
- net +3.3V: now also TP6.1
- net GND: now also TP5.1
- net 485_LED+ renamed 485_LED1_+
- net 485_LED1_+: no longer J6.2 (Pin_2)
- net 485_LED- renamed 485_LED1_-
- net 485_LED1_-: no longer J6.3 (Pin_3)
- new net 485_LED2_+: J6.2 (Pin_2)
- new net 485_LED2_-: J6.3 (Pin_3)
Other:
- sheet MCU_ESP32 ports: added 485_LED1_A, 485_LED1_B, 485_LED2_A, 485_LED2_B; removed 12V_SE, 24V_SE, 485_LED_A, 485_LED_B

Commit message: HUB Hardware V1.1.0
Parts:
- removed C1: 33uF 35V, easyeda2kicad:CAP-SMD_BD6.3-L6.6-W6.6-FD, symbol easyeda2kicad:RVT1V330M0605_c27784
- removed J2: Conn_01x03, Connector_JST:JST_VH_B3P-VH_1x03_P3.96mm_Vertical, symbol Connector_Generic:Conn_01x03
- added C1: 22uF 35V, Capacitor_SMD:C_1206_3216Metric, symbol Device:C
- added J2: Conn_01x01_Pin, Connector_Wire:SolderWire-0.75sqmm_1x01_D1.25mm_OD3.5mm, symbol Connector:Conn_01x01_Pin
- added J7: Conn_01x05, Connector_JST:JST_VH_B5P-VH-B_1x05_P3.96mm_Vertical, symbol Connector_Generic:Conn_01x05
- U1: value K7803M-1000R3_C2916516 -> K7803M-1000R3
Connections:
- net +12V: now also J2.1 (Pin_1)
- net +24V: now also C1.1, J7.1 (Pin_1), J7.2 (Pin_2)
- net 485_ROV+: now also J1.3 (Pin_3); no longer J1.7 (Pin_7)
- net 485_ROV-: now also J1.4 (Pin_4); no longer J1.8 (Pin_8)
- net ETH_BD3D_RX+: now also J4.6 (Pin_6); no longer J4.5 (Pin_5)
- net ETH_BD3D_RX-: now also J4.5 (Pin_5); no longer J4.4 (Pin_4)
- net ETH_BD3D_TX+: now also J4.3 (Pin_3); no longer J4.2 (Pin_2)
- net ETH_BD3D_TX-: now also J4.4 (Pin_4); no longer J4.3 (Pin_3)
- net ETH_ROV_RX+: now also J1.5 (Pin_5); no longer J1.3 (Pin_3)
- net ETH_ROV_RX-: now also J1.6 (Pin_6); no longer J1.4 (Pin_4)
- net ETH_ROV_TX+: now also J1.8 (Pin_8); no longer J1.6 (Pin_6)
- net ETH_ROV_TX-: now also J1.7 (Pin_7); no longer J1.5 (Pin_5)
- net EXPOSURE: now also J4.2 (Pin_2); no longer J4.6 (Pin_6)
- net GND: now also C1.2, J7.4 (Pin_4), J7.5 (Pin_5)
- net PWM_LIGHT: now also J7.3 (Pin_3)
