File: MPE_HUB_Board/HUB_MPE.kicad_sch (KiCad schematic)
At the start: 22 parts, among them J1 Conn_01x09, J2 Conn_01x01_Pin, J3 Conn_01x06, J4 Conn_01x07, J5 Conn_01x05, J6 Conn_01x05, J7 Conn_01x05, U1 K7803M-1000R3

Commit message: Update 18/07/2025
Connections:
- no-connect marks 8 -> 9
Other:
- sheet MCU_ESP32 ports: added none; removed ~{RESET_SWITCH}
Changed lines of the file:
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@@
 	)
 	(no_connect
+		(at 245.11 132.08)
+	)
+	(no_connect
 		(at 360.68 241.3)
 	)
@@
 	(wire
 		(pts
-			(xy 149.86 228.6) (xy 130.81 228.6)
-		)
-		(stroke
-			(width 0)
-			(type default)
-		)
-	)
-	(wire
-		(pts
 			(xy 71.12 38.1) (xy 74.93 38.1)
 		)
@@
 		)
 	)
-	(label "RESET_SWITCH"
-		(at 130.81 228.6 0)
-		(effects
-			(font
-				(size 1.27 1.27)
-			)
-			(justify left bottom)
-		)
-	)
 	(label "485_LED2_+"
 		(at 130.81 217.17 0)
@@
 		)
 	)
-	(label "RESET_SWITCH"
-		(at 245.11 132.08 180)
-		(effects
-			(font
-				(size 1.27 1.27)
-			)
-			(justify right bottom)
-		)
-	)
 	(label "+12V_MULTISENSE"
 		(at 130.81 173.99 0)
@@
 		(polyline
 			(pts
-				(xy 186.055 97.79) (xy 187.325 97.79) (xy 187.325 124.46) (xy 186.055 124.46)
+				(xy 227.965 97.79) (xy 229.235 97.79) (xy 229.235 124.46) (xy 227.965 124.46)
 			)
 			(stroke
@@
 		(polyline
 			(pts
-				(xy 227.965 97.79) (xy 229.235 97.79) (xy 229.235 124.46) (xy 227.965 124.46)
+				(xy 186.055 97.79) (xy 187.325 97.79) (xy 187.325 124.46) (xy 186.055 124.46)
 			)
 			(stroke
@@
 			(effects
 				(font
-					(size 1.27 1.27)
-				)
-				(justify left)
-			)
-		)
-		(pin "~{RESET_SWITCH}" output
-			(at 149.86 228.6 180)
-			(effects
-				(font

Commit message: update 28/07/2025
Parts:
- removed U1: K7803M-1000R3, easyeda2kicad:PWRM-TH_DEXU_K78XXM-1000R3_XXXXXX, symbol easyeda2kicad:K7803M-1000R3_C2916516
Other:
- added sheet PSU_3V3 (PSU_3V3.kicad_sch)
- moved on the sheet: TP5, TP6

Commit message: Update 08/08/2025
Parts:
- removed C1: 22uF 35V, Capacitor_SMD:C_1206_3216Metric, symbol Device:C
- removed C3: 22uF 10V, Capacitor_SMD:C_0603_1608Metric, symbol Device:C
- LED2: LCSC (none) -> C2296
Other:
- moved on the sheet: C2, TP4, TP5
