File: MPE_HUB_Board/Switch_Ethernet_RTL8305NB.kicad_sch (KiCad schematic)
At the start: 68 parts, among them T1 H1102NLT, T2 H1102NLT, T3 H1102NLT, T4 H1102NLT, T5 H1102NLT, U2 RTL8305NB-VB-CG, X1 25Mhz

Commit message: Risolto problema reset (Nel firmware V2)
Other:
- company: (none) -> 3DResearch
- title: (none) -> Switch_Ethernet_RTL8305NB
Changed lines of the file:
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@@
 	(generator_version "9.0")
 	(paper "A4")
+	(title_block
+		(title "Switch_Ethernet_RTL8305NB")
+		(date "2025-03-21")
+		(rev "1.0")
+		(company "3DResearch")
+	)
 	(junction
 		(at 120.65 21.59)
@@
 		(polyline
 			(pts
-				(xy 125.73 154.305) (xy 125.73 153.035) (xy 157.48 153.035) (xy 157.48 154.305)
+				(xy 109.855 95.25) (xy 111.125 95.25) (xy 111.125 129.54) (xy 109.855 129.54)
 			)
 			(stroke
@@
 		(polyline
 			(pts
-				(xy 109.855 95.25) (xy 111.125 95.25) (xy 111.125 129.54) (xy 109.855 129.54)
+				(xy 125.73 154.305) (xy 125.73 153.035) (xy 157.48 153.035) (xy 157.48 154.305)
 			)
 			(stroke
