File: MPE_HUB_Board/W5500 - Eth.kicad_sch (KiCad schematic)
At the start: 61 parts, among them T6 H1102NLT, U7 W5500, X2 25MHz

Commit message: Risolto problema reset (Nel firmware V2)
Other:
- company: (none) -> 3DResearch
- title: (none) -> W5500 SPI ETH
Changed lines of the file:
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@@
 	(generator_version "9.0")
 	(paper "A4")
+	(title_block
+		(title "W5500 SPI ETH")
+		(date "2025-03-21")
+		(rev "1.0")
+		(company "3DResearch")
+	)
 	(rectangle
 		(start 17.78 57.15)

Commit message: HUB Hardware V1.1.0
Parts:
- TP1, TP2, TP3: footprint TestPoint:TestPoint_Pad_D3.0mm -> TestPoint:TestPoint_Pad_D1.0mm
Changed lines of the file:
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@@
 			)
 		)
-		(property "Footprint" "TestPoint:TestPoint_Pad_D3.0mm"
+		(property "Footprint" "TestPoint:TestPoint_Pad_D1.0mm"
 			(at 173.99 111.76 0)
 			(effects
@@
 			)
 		)
-		(property "Footprint" "TestPoint:TestPoint_Pad_D3.0mm"
+		(property "Footprint" "TestPoint:TestPoint_Pad_D1.0mm"
 			(at 127 104.14 0)
 			(effects
@@
 			)
 		)
-		(property "Footprint" "TestPoint:TestPoint_Pad_D3.0mm"
+		(property "Footprint" "TestPoint:TestPoint_Pad_D1.0mm"
 			(at 123.19 88.9 0)
 			(effects
