File: MPE_HUB_Board/MCU_ESP32.kicad_sch (KiCad schematic)
At the start: 76 parts, among them Q1 IRLML0100TRPBF, U10 MAX3485ESA, U11 AMS1117-3.3, U3 MAX3485ESA, U4 ESP32-S3-MINI-1-N4R2, U8 MAX3485ESA, U9 ADS1015IDGSR

Commit message: Update 18/07/2025
Parts:
- removed D1: 1N4148W T4, easyeda2kicad:SOD-123_L2.8-W1.8-LS3.7-RD, symbol easyeda2kicad:1N4148WT4
- removed U10, U3, U8: MAX3485ESA, easyeda2kicad:SOP-8_L5.0-W4.0-P1.27-LS6.0-BL, symbol easyeda2kicad:MAX3485ESA
- added C74, C75, C76: 3.3nF, Capacitor_SMD:C_0603_1608Metric, symbol jlcpcb_parts:CC0603KRX7R9BB104
- added C77: 1.8nF, Capacitor_SMD:C_0603_1608Metric, symbol jlcpcb_parts:CC0603KRX7R9BB104
- added D1, D4, D5: 1N4148W, easyeda2kicad:SOD-123F_L2.7-W1.6-LS3.8-RD, symbol jlcpcb_parts:1N4148W_C81598
- added R110: 220, Resistor_SMD:R_0603_1608Metric, symbol Device:R
- added R112: 560K, easyeda2kicad:R0603, symbol Device:R
- added R113: 1M, easyeda2kicad:R0603, symbol Device:R
- added U10, U12, U3: SN65HVD72DR, easyeda2kicad:SOP-8_L5.0-W4.0-P1.27-LS6.0-BL, symbol easyeda2kicad:SN65HVD72DR
- added U8: CD4093BM, easyeda2kicad:SOIC-14_L8.7-W3.9-P1.27-LS6.0-BL, symbol jlcpcb_parts:CD4093BM
Connections:
- net 3V3_MCU: now also U10.8 (VCC), U12.8 (VCC), U3.8 (VCC), U8.1 (A)
- net BUZZ: now also R110.2; no longer Q1.1 (G)
- net GND_MCU: now also C76.1, C77.1, D4.2 (A), R113.2, U10.5 (GND), U12.5 (GND), U3.5 (GND), U8.8 (E)
- net RX1_485_ROV: now also U12.1 (RO)
- net RX2_485_LED1: now also U10.1 (RO)
- net RX3_485_LED2: now also U3.1 (RO)
- net R/W_485_LED1: now also U10.2 (~{RE}), U10.3 (DE)
- net R/W_485_LED2: now also U3.2 (~{RE}), U3.3 (DE)
- net R/W_485_ROV: now also U12.2 (~{RE}), U12.3 (DE)
- net TX1_485_ROV: now also U12.4 (DI)
- net TX2_485_LED1: now also U10.4 (DI)
- net TX3_485_LED2: now also U3.4 (DI)
- net at R109.1: now also U12.6 (A)
- net at R108.1: now also U12.7 (B)
- net at R31.1: now also U3.6 (A)
- net at R26.1: now also U3.7 (B)
- net at BUZZER1.1 (+), R36.2: now also D1.1 (K)
- net at BUZZER1.2, Q1.3 (D): now also D1.2 (A)
- net at R94.1: now also U10.6 (A)
- net at R93.1: now also U10.7 (B)
- net ~{RESET_SWITCH} renamed WATER_PROBE
- net WATER_PROBE: now also U8.5 (C)
- new net: Q1.1 (G), R110.1
- new net: C74.1, D4.1 (K), D5.2 (A)
- new net: C76.2, D5.1 (K), R113.1, U8.10 (L), U8.9 (F)
- new net: U8.11 (M), U8.6 (D), U8.7 (VSS)
- new net: C75.2, R112.1, U8.12 (G)
- new net: C77.2, R112.2, U8.13 (H), U8.14 (VDD)
- new net DOWNTRACE_WATER: C74.2
- new net UPTRACE_WATER: C75.1
- no-connect marks 11 -> 16

Commit message: Update 08/08/2025
Parts:
- removed C43: 22uF, Capacitor_SMD:C_0603_1608Metric, symbol easyeda2kicad:CL31A226KAHNNNE
- added C43: 22uF 25V, Capacitor_SMD:C_0805_2012Metric, symbol Kicad_JLCPCB_Library:CL21A226MAQNNNE
- C74, C75, C76: LCSC (none) -> C1613
- C77: LCSC (none) -> C1599
- D1, D4, D5: LCSC (none) -> C81598
- R108, R109, R26, R31, R93, R94: LCSC (none) -> C844519
- R112: LCSC (none) -> C23203
- R113: LCSC (none) -> C2907115
- R37, R38: LCSC (none) -> C23186
- U10, U12, U3: LCSC (none) -> C48125
- U8: LCSC (none) -> C160714
- U9: LCSC (none) -> C193969
- USB2: LCSC (none) -> C720628
Connections:
- net 3V3_MCU: now also U8.14 (VDD), C43.2; no longer U8.1 (A)
- net GND_MCU: now also U8.7 (VSS), C43.1; no longer U8.8 (E)
- net WATER_PROBE: now also U8.10 (L); no longer U8.5 (C)
- net at C76.2, D5.1 (K), R113.1: now also U8.5 (C), U8.6 (D); no longer U8.10 (L), U8.9 (F)
- net at C75.2, R112.1: now also U8.3 (J); no longer U8.12 (G)
- net at C77.2, R112.2: now also U8.1 (A), U8.2 (B); no longer U8.13 (H), U8.14 (VDD)
- net at U8.4 (K): now also U8.8 (E), U8.9 (F)
- now unconnected: U8.11 (M)
