File: MPE_HUB_Board/PSU_3V3.kicad_sch (KiCad schematic)
At the start: 8 parts, among them U13 AP63203WU-7

Commit message: Update 08/08/2025
Parts:
- C78, C80: LCSC (none) -> C14663
- C79: LCSC (none) -> C194427
- C81: LCSC (none) -> C45783
- D6: footprint Kicad_JLCPCB_Library:SMA_L4.4-W2.8-LS5.4-R-RD -> easyeda2kicad:SMA_L4.4-W2.8-LS5.4-R-RD; LCSC (none) -> C22452
- L1: footprint Kicad_JLCPCB_Library:IND-SMD_L5.4-W5.2 -> easyeda2kicad:IND-SMD_L5.4-W5.2; LCSC (none) -> C408347
- U13: footprint Kicad_JLCPCB_Library:TSOT-26_L2.9-W1.6-P0.95-LS2.8-BL -> easyeda2kicad:TSOT-26_L2.9-W1.6-P0.95-LS2.8-BL; LCSC (none) -> C780769
Changed lines of the file:
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@@
 			)
 		)
-		(property "Footprint" "Kicad_JLCPCB_Library:IND-SMD_L5.4-W5.2"
+		(property "Footprint" "easyeda2kicad:IND-SMD_L5.4-W5.2"
 			(at 162.56 105.41 0)
 			(effects
@@
 		(property "LCSC Part" "C408347"
 			(at 162.56 110.49 0)
+			(effects
+				(font
+					(size 1.27 1.27)
+				)
+				(hide yes)
+			)
+		)
+		(property "LCSC" "C408347"
+			(at 162.56 91.44 0)
 			(effects
 				(font
@@
 			)
 		)
+		(property "LCSC" "C14663"
+			(at 140.97 93.345 0)
+			(effects
+				(font
+					(size 1.27 1.27)
+				)
+				(hide yes)
+			)
+		)
 		(pin "1"
 		)
@@
 			)
 		)
-		(property "Footprint" "Kicad_JLCPCB_Library:TSOT-26_L2.9-W1.6-P0.95-LS2.8-BL"
+		(property "Footprint" "easyeda2kicad:TSOT-26_L2.9-W1.6-P0.95-LS2.8-BL"
 			(at 124.46 107.95 0)
 			(effects
@@
 		(property "LCSC Part" "C780769"
 			(at 124.46 110.49 0)
+			(effects
+				(font
+					(size 1.27 1.27)
+				)
+				(hide yes)
+			)
+		)
+		(property "LCSC" "C780769"
+			(at 124.46 87.63 0)
 			(effects
 				(font
@@
 			)
 		)
+		(property "LCSC" "C14663"
+			(at 109.474 106.426 0)
+			(effects
+				(font
+					(size 1.27 1.27)
+				)
+				(hide yes)
+			)
+		)
 		(pin "1"
 		)
@@
 			)
 		)
+		(property "LCSC" "C194427"
+			(at 97.536 106.172 0)
+			(effects
+				(font
+					(size 1.27 1.27)
+				)
+				(hide yes)
+			)
+		)
 		(pin "2"
 		)
@@
 			)
 		)
-		(property "Footprint" "Kicad_JLCPCB_Library:SMA_L4.4-W2.8-LS5.4-R-RD"
+		(property "Footprint" "easyeda2kicad:SMA_L4.4-W2.8-LS5.4-R-RD"
 			(at 87.63 92.71 0)
 			(effects
@@
 		(property "LCSC Part" "C22452"
 			(at 87.63 87.63 0)
+			(effects
+				(font
+					(size 1.27 1.27)
+				)
+				(hide yes)
+			)
+		)
+		(property "LCSC" "C22452"
+			(at 90.17 104.14 0)
 			(effects
 				(font
@@
 			(effects
 				(font
+					(size 1.27 1.27)
+				)
+				(hide yes)
+			)
+		)
+		(property "LCSC" "C45783"
+			(at 175.26 107.9499 0)
+			(effects
+				(font
